Commit message: joint state publisher, first leg in rviz

File: src/sixlg_description/description/left_leg.urdf.xacro (robot description, xacro)
@@ -58,6 +58,6 @@
             <parent link="${name}/j1_link"/>
             <child link="${name}/j2_link"/>
-            <origin xyz="${femur_length} 0 0" rpy="0 -${pi} 0"/>
-            <axis xyz="0 1 0"/>
+            <origin xyz="${femur_length} 0 0" rpy="0 0 0"/>
+            <axis xyz="0 -1 0"/>
             <limit lower="0" upper="${pi}" velocity="100" effort="100"/>
         </joint>

Commit message: right leg urdf

File: src/sixlg_description/description/left_leg.urdf.xacro (robot description, xacro)
@@ -50,5 +50,5 @@
                 </geometry>
             </collision>
-            <xacro:inertial_box mass="0.1" x="${femur_length}" y="0" z="0">
+            <xacro:inertial_box mass="0.1" x="${femur_length}" y="0.01" z="0.002">
                 <origin xyz="${femur_length/2} 0 0" rpy="${pi/2} 0 0"/>
             </xacro:inertial_box>
@@ -70,4 +70,13 @@
                 <material name="blue"/>
             </visual>
+            <collision>
+                <origin xyz="${tibia_length/2} 0 0" rpy="${pi/2} 0 0"/>
+                <geometry>
+                    <box size="${tibia_length} 0.007 0.002"/>
+                </geometry>
+            </collision>
+            <xacro:inertial_box mass="0.1" x="${tibia_length}" y="0.007" z="0.002">
+                <origin xyz="${tibia_length/2} 0 0" rpy="${pi/2} 0 0"/>
+            </xacro:inertial_box>
         </link>
     </xacro:macro>

File: src/sixlg_description/description/robot_core.urdf.xacro (robot description, xacro)
@@ -5,4 +5,5 @@
     <xacro:include filename="materials.urdf.xacro"/>
     <xacro:include filename="left_leg.urdf.xacro"/>
+    <xacro:include filename="right_leg.urdf.xacro"/>
     <!-- CONSTANTS -->
     <xacro:property name="body_length" value="0.16"/>
@@ -45,3 +46,6 @@
             <origin xyz="0 ${body_width/2} 0" rpy="0 0 0"/>
     </xacro:left_leg>
+    <xacro:right_leg name="leg1" parent="body_link">
+            <origin xyz="0 -${body_width/2} 0" rpy="0 0 ${pi}"/>
+    </xacro:right_leg>
 </robot>
