Commit message: urdf done

File: src/sixlg_description/description/robot_core.urdf.xacro (robot description, xacro)
@@ -12,4 +12,5 @@
     <xacro:property name="femur_length" value="0.08"/>
     <xacro:property name="tibia_length" value="0.12"/>
+    <xacro:property name="front_leg_angle" value="${pi/4}"/>
     <!-- BASE LINK -->
     <link name="base_link">
@@ -43,9 +44,21 @@
     </gazebo>
     <!-- LEGS -->
-    <xacro:left_leg name="leg0" parent="body_link">
-            <origin xyz="0 ${body_width/2} 0" rpy="0 0 0"/>
-    </xacro:left_leg>
+    <xacro:right_leg name="leg0" parent="body_link">
+            <origin xyz="${body_length/2} -${body_width/2} 0" rpy="0 0 ${pi + front_leg_angle}"/>
+    </xacro:right_leg>
     <xacro:right_leg name="leg1" parent="body_link">
             <origin xyz="0 -${body_width/2} 0" rpy="0 0 ${pi}"/>
     </xacro:right_leg>
+    <xacro:right_leg name="leg2" parent="body_link">
+            <origin xyz="-${body_length/2} -${body_width/2} 0" rpy="0 0 ${pi - front_leg_angle}"/>
+    </xacro:right_leg>
+    <xacro:left_leg name="leg3" parent="body_link">
+            <origin xyz="-${body_length/2} ${body_width/2} 0" rpy="0 0 ${front_leg_angle}"/>
+    </xacro:left_leg>
+    <xacro:left_leg name="leg4" parent="body_link">
+            <origin xyz="0 ${body_width/2} 0" rpy="0 0 0"/>
+    </xacro:left_leg>
+    <xacro:left_leg name="leg5" parent="body_link">
+            <origin xyz="${body_length/2} ${body_width/2} 0" rpy="0 0 -${front_leg_angle}"/>
+    </xacro:left_leg>
 </robot>

Commit message: walking in simulation

File: src/sixlg_description/description/robot_core.urdf.xacro (robot description, xacro)
@@ -12,5 +12,5 @@
     <xacro:property name="femur_length" value="0.08"/>
     <xacro:property name="tibia_length" value="0.12"/>
-    <xacro:property name="front_leg_angle" value="${pi/4}"/>
+    <xacro:property name="angle_to_font" value="${pi/4}"/>
     <!-- BASE LINK -->
     <link name="base_link">
@@ -45,5 +45,5 @@
     <!-- LEGS -->
     <xacro:right_leg name="leg0" parent="body_link">
-            <origin xyz="${body_length/2} -${body_width/2} 0" rpy="0 0 ${pi + front_leg_angle}"/>
+            <origin xyz="${body_length/2} -${body_width/2} 0" rpy="0 0 ${pi + angle_to_font}"/>
     </xacro:right_leg>
     <xacro:right_leg name="leg1" parent="body_link">
@@ -51,8 +51,8 @@
     </xacro:right_leg>
     <xacro:right_leg name="leg2" parent="body_link">
-            <origin xyz="-${body_length/2} -${body_width/2} 0" rpy="0 0 ${pi - front_leg_angle}"/>
+            <origin xyz="-${body_length/2} -${body_width/2} 0" rpy="0 0 ${pi - angle_to_font}"/>
     </xacro:right_leg>
     <xacro:left_leg name="leg3" parent="body_link">
-            <origin xyz="-${body_length/2} ${body_width/2} 0" rpy="0 0 ${front_leg_angle}"/>
+            <origin xyz="-${body_length/2} ${body_width/2} 0" rpy="0 0 ${angle_to_font}"/>
     </xacro:left_leg>
     <xacro:left_leg name="leg4" parent="body_link">
@@ -60,5 +60,5 @@
     </xacro:left_leg>
     <xacro:left_leg name="leg5" parent="body_link">
-            <origin xyz="${body_length/2} ${body_width/2} 0" rpy="0 0 -${front_leg_angle}"/>
+            <origin xyz="${body_length/2} ${body_width/2} 0" rpy="0 0 -${angle_to_font}"/>
     </xacro:left_leg>
 </robot>
